File: examples/can-interface-reference/Reforge_CAN_Interface_Reference.kicad_pcb (KiCad board)
At the start: 2 copper layers, 60 x 42 mm, 10 parts, among them J1 CAN / 12V INPUT, J2 REFORGE EXPANSION, U1 MCP1799T-3302H/TT, U2 SN65HVD230D

Commit message: Fix CAN reference fabrication and 3D models
Parts:
- C1: footprint Reforge_Reference:C1 -> C1
- C2: footprint Reforge_Reference:C2 -> C2
- C3: footprint Reforge_Reference:C3 -> C3
- J1: footprint Reforge_Reference:J1 -> J1
- J2: footprint Reforge_Reference:J2 -> J2
- JP1: footprint Reforge_Reference:JP1 -> JP1
- R1: footprint Reforge_Reference:R1 -> R1
- R2: footprint Reforge_Reference:R2 -> R2
- U1: footprint Reforge_Reference:U1 -> U1
Changed lines of the file:
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@@
   (net 7 "TX_IDLE")
   (net 8 "TERM_MID")
-  (footprint "Reforge_Reference:J1"
+  (footprint "J1"
     (layer "F.Cu") (at 103.00 104.00 0)
         (property "Reference" "J1"
@@
     )
     (attr through_hole)
-    (fp_rect (start -3.00 -10.00) (end 3.00 10.00)
+    (fp_rect (start -3.00 -2.38) (end 3.00 17.62)
       (stroke (width 0.20) (type default)) (fill none) (layer "F.Fab") )
     (pad "1" thru_hole rect (at 0.00 0.00) (size 3.20 3.20) (drill 1.30) (layers "*.Cu" "*.Mask")
@@
     (pad "4" thru_hole circle (at 0.00 15.24) (size 3.20 3.20) (drill 1.30) (layers "*.Cu" "*.Mask")
       (net 4 "GND") (pinfunction "4") (pintype "passive") )
-  )
-  (footprint "Reforge_Reference:J2"
+    (model "${KICAD10_3DMODEL_DIR}/TerminalBlock_Phoenix.3dshapes/TerminalBlock_Phoenix_MKDS-1,5-4-5.08_1x04_P5.08mm_Horizontal.step"
+      (offset (xyz 0 0 0))
+      (scale (xyz 1 1 1))
+      (rotate (xyz 0 0 90))
+    ))
+  (footprint "J2"
     (layer "F.Cu") (at 157.00 105.00 0)
         (property "Reference" "J2"
@@
     )
     (attr through_hole)
-    (fp_rect (start -1.90 -5.10) (end 1.90 5.10)
+    (fp_rect (start -1.90 -1.29) (end 1.90 8.91)
       (stroke (width 0.20) (type default)) (fill none) (layer "F.Fab") )
     (pad "1" thru_hole rect (at 0.00 0.00) (size 2.00 2.00) (drill 1.00) (layers "*.Cu" "*.Mask")
@@
     (pad "4" thru_hole circle (at 0.00 7.62) (size 2.00 2.00) (drill 1.00) (layers "*.Cu" "*.Mask")
       (net 4 "GND") (pinfunction "4") (pintype "passive") )
-  )
-  (footprint "Reforge_Reference:JP1"
+    (model "${KICAD10_3DMODEL_DIR}/Connector_PinHeader_2.54mm.3dshapes/PinHeader_1x04_P2.54mm_Vertical.step"
+      (offset (xyz 0 0 0))
+      (scale (xyz 1 1 1))
+      (rotate (xyz 0 0 0))
+    ))
+  (footprint "JP1"
     (layer "F.Cu") (at 119.00 102.00 0)
         (property "Reference" "JP1"
@@
     (pad "2" thru_hole circle (at 2.54 0.00) (size 2.20 2.20) (drill 1.00) (layers "*.Cu" "*.Mask")
       (net 1 "CAN_L") (pinfunction "2") (pintype "passive") )
-  )
-  (footprint "Reforge_Reference:U1"
+    (model "${KICAD10_3DMODEL_DIR}/Connector_PinHeader_2.54mm.3dshapes/PinHeader_1x02_P2.54mm_Vertical.step"
+      (offset (xyz 0 0 0))
+      (scale (xyz 1 1 1))
+      (rotate (xyz 0 0 -90))
+    ))
+  (footprint "U1"
     (layer "F.Cu") (at 120.00 124.00 0)
         (property "Reference" "U1"
@@
     (pad "3" smd roundrect (at 0.95 0.00) (size 1.10 1.40) (layers "F.Cu" "F.Paste" "F.Mask") (roundrect_rratio 0.25)
       (net 3 "+12V") (pinfunction "3") (pintype "passive") )
-  )
+    (model "${KICAD10_3DMODEL_DIR}/Package_TO_SOT_SMD.3dshapes/SOT-23-3.step"
+      (offset (xyz 0 0 0))
+      (scale (xyz 1 1 1))
+      (rotate (xyz 0 0 0))
+    ))
   (footprint "U2"
     (layer "F.Cu") (at 132.00 110.00 180)
@@
     (pad "8" smd roundrect (at 2.48 -1.91) (size 1.95 0.60) (layers "F.Cu" "F.Paste" "F.Mask") (roundrect_rratio 0.25)
       (net 4 "GND") (pinfunction "8") (pintype "passive") )
-  )
-  (footprint "Reforge_Reference:R1"
+    (model "${KICAD10_3DMODEL_DIR}/Package_SO.3dshapes/SOIC-8_3.9x4.9mm_P1.27mm.step"
+      (offset (xyz 0 0 0))
+      (scale (xyz 1 1 1))
+      (rotate (xyz 0 0 0))
+    ))
+  (footprint "R1"
     (layer "F.Cu") (at 148.00 126.00 0)
         (property "Reference" "R1"
@@
     (pad "2" smd roundrect (at 1.00 0.00) (size 1.20 1.40) (layers "F.Cu" "F.Paste" "F.Mask") (roundrect_rratio 0.25)
       (net 7 "TX_IDLE") (pinfunction "2") (pintype "passive") )
-  )
-  (footprint "Reforge_Reference:R2"
+    (model "${KICAD10_3DMODEL_DIR}/Resistor_SMD.3dshapes/R_0805_2012Metric.step"
+      (offset (xyz 0 0 0))
+      (scale (xyz 1 1 1))
+      (rotate (xyz 0 0 0))
+    ))
+  (footprint "R2"
     (layer "F.Cu") (at 115.00 102.00 0)
         (property "Reference" "R2"
@@
     (pad "2" smd roundrect (at 1.00 0.00) (size 1.20 1.40) (layers "F.Cu" "F.Paste" "F.Mask") (roundrect_rratio 0.25)
       (net 8 "TERM_MID") (pinfunction "2") (pintype "passive") )
-  )
-  (footprint "Reforge_Reference:C1"
+    (model "${KICAD10_3DMODEL_DIR}/Resistor_SMD.3dshapes/R_0805_2012Metric.step"
+      (offset (xyz 0 0 0))
+      (scale (xyz 1 1 1))
+      (rotate (xyz 0 0 0))
+    ))
+  (footprint "C1"
     (layer "F.Cu") (at 112.00 128.00 0)
         (property "Reference" "C1"
@@
     (pad "2" smd roundrect (at 1.00 0.00) (size 1.20 1.40) (layers "F.Cu" "F.Paste" "F.Mask") (roundrect_rratio 0.25)
       (net 4 "GND") (pinfunction "2") (pintype "passive") )
-  )
-  (footprint "Reforge_Reference:C2"
+    (model "${KICAD10_3DMODEL_DIR}/Capacitor_SMD.3dshapes/C_0805_2012Metric.step"
+      (offset (xyz 0 0 0))
+      (scale (xyz 1 1 1))
+      (rotate (xyz 0 0 0))
+    ))
+  (footprint "C2"
     (layer "F.Cu") (at 126.00 132.00 0)
         (property "Reference" "C2"
@@
     (pad "2" smd roundrect (at 1.00 0.00) (size 1.20 1.40) (layers "F.Cu" "F.Paste" "F.Mask") (roundrect_rratio 0.25)
       (net 4 "GND") (pinfunction "2") (pintype "passive") )
-  )
-  (footprint "Reforge_Reference:C3"
+    (model "${KICAD10_3DMODEL_DIR}/Capacitor_SMD.3dshapes/C_0805_2012Metric.step"
+      (offset (xyz 0 0 0))
+      (scale (xyz 1 1 1))
+      (rotate (xyz 0 0 0))
+    ))
+  (footprint "C3"
     (layer "F.Cu") (at 140.00 121.00 0)
         (property "Reference" "C3"
@@
     (pad "2" smd roundrect (at 1.00 0.00) (size 1.20 1.40) (layers "F.Cu" "F.Paste" "F.Mask") (roundrect_rratio 0.25)
       (net 4 "GND") (pinfunction "2") (pintype "passive") )
-  )
+    (model "${KICAD10_3DMODEL_DIR}/Capacitor_SMD.3dshapes/C_0805_2012Metric.step"
+      (offset (xyz 0 0 0))
+      (scale (xyz 1 1 1))
+      (rotate (xyz 0 0 0))
+    ))
   (gr_rect (start 100 98) (end 160 140) (stroke (width 0.25) (type default)) (fill none) (layer "Edge.Cuts") )
   (gr_text "UNTESTED REFERENCE ONLY" (at 130 138) (layer "F.SilkS") (effects (font (size 1.3 1.3) (thickness 0.22))) )

Commit message: Use Reforge JST GH connector on CAN reference
Parts:
- J2: value REFORGE EXPANSION -> JST GH SM04B-GHS-TB
- moved J2 1.89 mm to (156.8, 103.1), turned to 90 degrees
Routing:
- net GND: track 192.7 -> 209.0 mm, vias 6 -> 7
- net CAN_L: track 42.3 -> 34.5 mm
- net TX_IDLE: track 45.5 -> 50.9 mm, vias 0 -> 2
- net +12V: track 44.9 -> 41.9 mm
- net CAN_H: track 40.4 -> 38.1 mm
Other:
- board text added: "REFORGE ADV REV B"
- board text removed: "TO REFORGE ADV REV B"
